Commit message: Add files via upload

File: data/urdf_files/elfin5_l.urdf (robot description, URDF)
Before this commit: robot elfin5_l, 10 links, 9 joints
Links:
- removed link world
- link elfin_base: mass 0.68795 -> None; geometry 
- link elfin_base_link: geometry 
- link elfin_end_link: geometry 
- link elfin_link1: mass 2.5856 -> None; geometry 
- link elfin_link2: mass 1.208607 -> None; geometry 
- link elfin_link3: mass 1.5324 -> None; geometry 
- link elfin_link4: mass 0.5 -> None; geometry 
- link elfin_link5: mass 0.81192 -> None; geometry 
- link elfin_link6: mass 0.11343 -> None; geometry 
Joints:
- removed joint world_base
- joint elfin_end_joint: axis 0 0 0 -> (none)
- joint elfin_joint1: limit lower=-3.14 upper=3.14 effort=420 velocity=1.57 -> lower=-3.14 upper=3.14
- joint elfin_joint2: limit lower=-2.35 upper=2.35 effort=420 velocity=1.57 -> lower=-2.35 upper=2.35
- joint elfin_joint3: limit lower=-2.61 upper=2.61 effort=200 velocity=1.57 -> lower=-2.61 upper=2.61
- joint elfin_joint4: limit lower=-3.14 upper=3.14 effort=200 velocity=1.57 -> lower=-3.14 upper=3.14
- joint elfin_joint5: limit lower=-2.56 upper=2.56 effort=69 velocity=1.57 -> lower=-2.56 upper=2.56
- joint elfin_joint6: limit lower=-3.14 upper=3.14 effort=69 velocity=1.57 -> lower=-3.14 upper=3.14

Commit message: complete elfin5 URDF (inertial/collision/visual) and correct end_link geometry

File: data/urdf_files/elfin5_l.urdf (robot description, URDF)
Before this commit: robot elfin5_l, 9 links, 8 joints
Links:
- link elfin_base: mass None -> 0.68795; geometry collision mesh filename=../meshes/elfin_base.STL scale=1.2 1.2 1.2; visual mesh filename=../meshes/elfin_base.STL
- link elfin_base_link: geometry collision box size=0.001 0.001 0.001; visual box size=0.001 0.001 0.001
- link elfin_end_link: geometry collision box size=0.001 0.001 0.001; visual box size=0.0015 0.0015 0.0015
- link elfin_link1: mass None -> 2.5856; geometry collision mesh filename=../meshes/elfin_link1.STL scale=1.2 1.2 1.2; visual mesh filename=../meshes/elfin_link1.STL
- link elfin_link2: mass None -> 1.208607; geometry collision mesh filename=../meshes/elfin_link2.STL scale=1.2 1.2 1.2; visual mesh filename=../meshes/elfin_link2.STL
- link elfin_link3: mass None -> 1.5324; geometry collision mesh filename=../meshes/elfin_link3.STL scale=1.2 1.2 1.2; visual mesh filename=../meshes/elfin_link3.STL
- link elfin_link4: mass None -> 0.5; geometry collision mesh filename=../meshes/elfin_link4.STL scale=1.2 1.2 1.2; visual mesh filename=../meshes/elfin_link4.STL
- link elfin_link5: mass None -> 0.81192; geometry collision mesh filename=../meshes/elfin_link5.STL scale=1.2 1.2 1.2; visual mesh filename=../meshes/elfin_link5.STL
- link elfin_link6: mass None -> 0.11343; geometry collision mesh filename=../meshes/elfin_link6.STL scale=1.2 1.2 1.2; visual mesh filename=../meshes/elfin_link6.STL
Joints:
- joint elfin_joint1: limit lower=-3.14 upper=3.14 -> lower=-3.14 upper=3.14 effort=420 velocity=1.57
- joint elfin_joint2: limit lower=-2.35 upper=2.35 -> lower=-2.35 upper=2.35 effort=420 velocity=1.57
- joint elfin_joint3: limit lower=-2.61 upper=2.61 -> lower=-2.61 upper=2.61 effort=200 velocity=1.57
- joint elfin_joint4: limit lower=-3.14 upper=3.14 -> lower=-3.14 upper=3.14 effort=200 velocity=1.57
- joint elfin_joint5: limit lower=-2.56 upper=2.56 -> lower=-2.56 upper=2.56 effort=69 velocity=1.57
- joint elfin_joint6: limit lower=-3.14 upper=3.14 -> lower=-3.14 upper=3.14 effort=69 velocity=1.57
